File: 6.kicad_sch (KiCad schematic)
At the start: 1 part, among them J6 ERF8-025-05.0-L-DV-L-K-TR

Commit message: final setup for power rails
Connections:
- net 5V0_USB: now reaches J6.22
- net 5V0_USB: now also J6.24, J6.26, J6.28, J6.30
