File: 2.kicad_sch (KiCad schematic)
At the start: 1 part, among them J2 ERF8-025-05.0-L-DV-L-K-TR

Commit message: initialized for 4-card
Connections:
- net USB3.RX_N: now reaches J2.14
- net USB3.RX_P: now reaches J2.16
- net USB3.TX_N: now reaches J2.22
- net USB3.TX_P: now reaches J2.24
- net CMRF.MOSI: now reaches J2.30
- net CMRF.MISO: now reaches J2.32
- net CMRF.SCLK: now reaches J2.38
- net CMRF.CS0n: now reaches J2.40
- net USB3.D_N: now reaches J2.6
- net USB3.D_P: now reaches J2.8

Commit message: fixed footprint link
Connections:
- net CAN0.H: now also J2.03; no longer J2.3
- net CAN0.L: now also J2.01; no longer J2.1
- net GND: now also J2.02, J2.04, J2.05, J2.07; no longer J2.2, J2.4, J2.5, J2.7
- net USB3.D_N: now also J2.06; no longer J2.6
- net USB3.D_P: now also J2.08; no longer J2.8
Changed lines of the file:
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@@
 		(pin "10"
 		)
-		(pin "8"
+		(pin "01"
 		)
-		(pin "6"
+		(pin "03"
 		)
-		(pin "4"
+		(pin "05"
 		)
-		(pin "2"
+		(pin "07"
 		)
 		(pin "40"
@@
 		(pin "11"
 		)
-		(pin "9"
+		(pin "09"
 		)
-		(pin "7"
+		(pin "02"
 		)
-		(pin "5"
+		(pin "04"
 		)
-		(pin "3"
+		(pin "06"
 		)
-		(pin "1"
+		(pin "08"
 		)
 		(pin "33"

Commit message: added pwr leds and edge cuts
Connections:
- net CAN0.H renamed CAN0.P
- net CAN0.L renamed CAN0.N
Changed lines of the file:
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@@
+		)
+	)
+	(label "CAN0.P"
+		(at 102.87 71.12 0)
+		(effects
+			(font
+				(size 1.27 1.27)
+			)
+			(justify left bottom)
 		)
 	)
@@
 		)
 	)
-	(label "CAN0.L"
-		(at 102.87 68.58 0)
-		(effects
-			(font
-				(size 1.27 1.27)
-			)
-			(justify left bottom)
-		)
-	)
 	(label "CMRF.MISO"
 		(at 181.61 106.68 180)
@@
 		)
 	)
-	(label "CAN0.H"
-		(at 102.87 71.12 0)
+	(label "CAN0.N"
+		(at 102.87 68.58 0)
 		(effects
 			(font

Commit message: prelim layout complete
Connections:
- net 5V0: now also J2.02, J2.04, J2.06, J2.08, J2.10; no longer J2.41, J2.43, J2.45, J2.47, J2.49
- net CAN0.N: now also J2.50; no longer J2.01
- net CAN0.P: now also J2.48; no longer J2.03
- net CMRF.CS0n: now also J2.11; no longer J2.40
- net CMRF.MISO: now also J2.19; no longer J2.32
- net CMRF.MOSI: now also J2.21; no longer J2.30
- net CMRF.SCLK: now also J2.13; no longer J2.38
- net GND: now also J2.01, J2.09, J2.14, J2.17, J2.22, J2.25, J2.30, J2.33, J2.38, J2.41, J2.46, J2.47, J2.49; no longer J2.02, J2.04, J2.05, J2.10, J2.13, J2.18, J2.21, J2.26, J2.29, J2.34, J2.37, J2.42, J2.50
- net USB3.D_N: now also J2.45; no longer J2.06
- net USB3.D_P: now also J2.43; no longer J2.08
- net USB3.RX_N: now also J2.37; no longer J2.14
- net USB3.RX_P: now also J2.35; no longer J2.16
- net USB3.TX_N: now also J2.29; no longer J2.22
- net USB3.TX_P: now also J2.27; no longer J2.24
