File: 3.kicad_sch (KiCad schematic)
At the start: 1 part, among them J3 ERF8-025-05.0-L-DV-L-K-TR

Commit message: fixed footprint link
Connections:
- net CAN0.H: now also J3.03; no longer J3.3
- net CAN0.L: now also J3.01; no longer J3.1
- net GND: now also J3.02, J3.04, J3.05, J3.07; no longer J3.2, J3.4, J3.5, J3.7
Changed lines of the file:
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@@
 		(pin "10"
 		)
-		(pin "8"
+		(pin "09"
 		)
-		(pin "6"
+		(pin "07"
 		)
-		(pin "4"
+		(pin "05"
 		)
-		(pin "2"
+		(pin "03"
 		)
 		(pin "40"
@@
 		(pin "11"
 		)
-		(pin "9"
+		(pin "01"
 		)
-		(pin "7"
+		(pin "02"
 		)
-		(pin "5"
+		(pin "04"
 		)
-		(pin "3"
+		(pin "06"
 		)
-		(pin "1"
+		(pin "08"
 		)
 		(pin "33"

Commit message: added pwr leds and edge cuts
Connections:
- net CAN0.H renamed CAN0.P
- net CAN0.L renamed CAN0.N
Changed lines of the file:
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@@
 		)
 	)
-	(label "CAN0.L"
+	(label "CAN0.N"
 		(at 102.87 68.58 0)
-		(effects
-			(font
-				(size 1.27 1.27)
-			)
-			(justify left bottom)
-		)
-	)
-	(label "CAN0.H"
-		(at 102.87 71.12 0)
 		(effects
 			(font
@@
 		)
 	)
+	(label "CAN0.P"
+		(at 102.87 71.12 0)
+		(effects
+			(font
+				(size 1.27 1.27)
+			)
+			(justify left bottom)
+		)
+	)

Commit message: prelim layout complete
Connections:
- net 5V0: now also J3.02, J3.04, J3.06, J3.08, J3.10; no longer J3.41, J3.43, J3.45, J3.47, J3.49
- net CAN0.N: now also J3.50; no longer J3.01
- net CAN0.P: now also J3.48; no longer J3.03
- net GND: now also J3.01, J3.09, J3.14, J3.17, J3.22, J3.25, J3.30, J3.33, J3.38, J3.41, J3.46, J3.47, J3.49; no longer J3.02, J3.04, J3.05, J3.10, J3.13, J3.18, J3.21, J3.26, J3.29, J3.34, J3.37, J3.42, J3.50
