File: 4.kicad_sch (KiCad schematic)
At the start: 1 part, among them J4 ERF8-025-05.0-L-DV-L-K-TR

Commit message: initialized for 4-card
Connections:
- net CMRF.MOSI: now reaches J4.38
- net CMRF.MISO: now reaches J4.40
- net CMRF.SCLK: now reaches J4.46
- net CMRF.CS0n: now reaches J4.48

Commit message: fixed footprint link
Connections:
- net CAN0.H: now also J4.03; no longer J4.3
- net CAN0.L: now also J4.01; no longer J4.1
- net CMRF.CS0n: now also J4.40; no longer J4.48
- net CMRF.MISO: now also J4.32; no longer J4.40
- net CMRF.MOSI: now also J4.30; no longer J4.38
- net CMRF.SCLK: now also J4.38; no longer J4.46
- net GND: now also J4.02, J4.04, J4.05, J4.07; no longer J4.2, J4.4, J4.5, J4.7

Commit message: added pwr leds and edge cuts
Connections:
- net CAN0.H renamed CAN0.P
- net CAN0.L renamed CAN0.N
Changed lines of the file:
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@@
 		)
 	)
-	(label "CAN0.L"
-		(at 102.87 68.58 0)
+	(label "CAN0.P"
+		(at 102.87 71.12 0)
 		(effects
 			(font
@@
 		)
 	)
+	(label "CAN0.N"
+		(at 102.87 68.58 0)
+		(effects
+			(font
+				(size 1.27 1.27)
+			)
+			(justify left bottom)
+		)
+	)
 	(label "CMRF.SCLK"
 		(at 181.61 114.3 180)
@@
 		)
 	)
-	(label "CAN0.H"
-		(at 102.87 71.12 0)
-		(effects
-			(font
-				(size 1.27 1.27)
-			)
-			(justify left bottom)
-		)
-	)

Commit message: prelim layout complete
Connections:
- net 5V0: now also J4.02, J4.04, J4.06, J4.08, J4.10; no longer J4.41, J4.43, J4.45, J4.47, J4.49
- net CAN0.N: now also J4.50; no longer J4.01
- net CAN0.P: now also J4.48; no longer J4.03
- net CMRF.CS0n: now also J4.11; no longer J4.40
- net CMRF.MISO: now also J4.19; no longer J4.32
- net CMRF.MOSI: now also J4.21; no longer J4.30
- net CMRF.SCLK: now also J4.13; no longer J4.38
- net GND: now also J4.01, J4.09, J4.14, J4.17, J4.22, J4.25, J4.30, J4.33, J4.38, J4.41, J4.46, J4.47, J4.49; no longer J4.02, J4.04, J4.05, J4.10, J4.13, J4.18, J4.21, J4.26, J4.29, J4.34, J4.37, J4.42, J4.50
