File: sch/lemon.kicad_sch (KiCad schematic)
At the start: 7 parts, among them J2 ERF8-025-05.0-L-DV-L-K-TR

Commit message: moved connectors, added silkscreen
Parts:
- removed GND2, GND3: TestPoint, library:KEYSTONE_575-4, symbol Connector:TestPoint

Commit message: rev b, flipped connectors
Connections:
- net 5VBUS1: now also J2.06, J2.08, J2.10, J2.12; no longer J2.39, J2.41, J2.43, J2.45
- net 5VBUS2: now also J2.18, J2.20, J2.22, J2.24; no longer J2.27, J2.29, J2.31, J2.33
- net 5VBUS3: now also J2.30, J2.32, J2.34, J2.36; no longer J2.15, J2.17, J2.19, J2.21
- net CAN0.N: now also J2.01; no longer J2.50
- net CAN0.P: now also J2.03; no longer J2.48
- net GND: now also J2.15, J2.17, J2.19, J2.21, J2.27, J2.29, J2.31, J2.33, J2.39, J2.41, J2.43, J2.45, J2.48, J2.50; no longer J2.01, J2.03, J2.06, J2.08, J2.10, J2.12, J2.18, J2.20, J2.22, J2.24, J2.30, J2.32, J2.34, J2.36
Other:
- moved on the sheet: J2
Changed lines of the file:
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@@
 	(symbol
 		(lib_id "library:ERF8-025-05.0-L-DV-L-K-TR")
-		(at 143.51 99.06 0)
+		(at 143.51 99.06 180)
 		(unit 1)
 		(body_style 1)
@@
 		(in_pos_files yes)
 		(dnp no)
-		(fields_autoplaced yes)
 		(property "Reference" "J2"
 			(at 143.51 60.96 0)
